File: pcb/draft_1-2/pcb/_autosave-pcb.kicad_pcb (KiCad board)
At the start: 2 copper layers, 29.5 x 39.4 mm, 28 parts, among them J1 USB4110-GF-A, J2 SWD, U1 H3LIS200DLTR, U2 ATSAML21J16B-AUT, U3 BQ25155

Commit message: add example image to readme
Parts:
- removed C11: 22uF, Capacitor_SMD:C_0805_2012Metric
- added TP1: GND, TestPoint:TestPoint_Pad_2.0x2.0mm, B.Cu at (133.1, 98.6)
- added TP2: 5V, TestPoint:TestPoint_Pad_2.0x2.0mm, B.Cu at (150.4, 98.6)
- added TP3: ~MR, TestPoint:TestPoint_Pad_2.0x2.0mm, B.Cu at (133.1, 103.6)
- added TP4: PMID, TestPoint:TestPoint_Pad_2.0x2.0mm, B.Cu at (150.4, 103.6)
- added TP5: 3V3, TestPoint:TestPoint_Pad_2.0x2.0mm, B.Cu at (150.4, 108.7)
- added TP6: 1V8, TestPoint:TestPoint_Pad_2.0x2.0mm, B.Cu at (150.4, 113.8)
- added TP7: SCL, TestPoint:TestPoint_Pad_2.0x2.0mm, B.Cu at (132.8, 113.8)
- added TP8: SDA, TestPoint:TestPoint_Pad_2.0x2.0mm, B.Cu at (133.1, 108.7)
- C1, C10, C2, C4, C5, C6, C7, C8, C9: footprint Capacitor_SMD:C_0402_1005Metric -> Capacitor_SMD:C_0805_2012Metric
- R1, R2, R3, R4, R5, R6, R7: footprint Resistor_SMD:R_0402_1005Metric -> Resistor_SMD:R_0805_2012Metric
- moved C4 4.28 mm to (140.7, 106.0)
- moved C5 3.49 mm to (132.2, 102.7)
- moved C3 3.05 mm to (132.2, 98.7)
- moved R3 2.68 mm to (150.6, 97.7)
- moved C1 2.54 mm to (147.2, 97.7), turned to 90 degrees
- moved U1 2.44 mm to (148.3, 101.5)
- moved U3 2.16 mm to (135.6, 102.2)
- moved C8 2.06 mm to (146.7, 124.2), turned to 180 degrees
- moved R4 2.04 mm to (144.3, 97.7)
- moved C2 1.76 mm to (139.7, 101.5), turned to 90 degrees
- moved C10 1.57 mm to (143.8, 101.6), turned to 90 degrees
- moved R7 1.57 mm to (132.2, 108.0), turned to 90 degrees
- moved R2 1.08 mm to (135.1, 108.0), turned to 90 degrees
- moved R5 1.02 mm to (146.1, 104.6), turned to 180 degrees
- moved R1 0.85 mm to (137.8, 108.0), turned to 90 degrees
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Connections:
- D1 pad 1: GND -> Net-(D1-Pad1)
- U2 pad 50: Net-(U2-Pad50) -> Net-(D1-Pad1)
Routing:
- net GND: track 143.5 -> 0.00 mm, vias 6 -> 0
- net +1V8: track 92.2 -> 0.00 mm, vias 2 -> 0
- net D+: track 33.6 -> 0.00 mm, vias 2 -> 0
- net D-: track 32.1 -> 0.00 mm, vias 2 -> 0
- net SDA: track 30.9 -> 0.00 mm, vias 3 -> 0
- net INT1: track 28.9 -> 0.00 mm, vias 2 -> 0
- net SCL: track 28.1 -> 0.00 mm, vias 3 -> 0
- net /1B: track 25.7 -> 0.00 mm
- net INT2: track 25.0 -> 0.00 mm, vias 2 -> 0
- net /1C: track 23.9 -> 0.00 mm
- net /1A: track 22.4 -> 0.00 mm
- net /1D: track 22.1 -> 0.00 mm
- net /1F: track 22.0 -> 0.00 mm
- net Net-(BT1-Pad1): track 20.6 -> 0.00 mm
- net /1E: track 20.3 -> 0.00 mm
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